File: accessControl.brd (EAGLE design)
At the start: 97.5 x 59.7 mm, 8 parts

Commit message: esp32 code
Connections:
- net N$1: now also U$1.GPIO32; no longer U$1.GPIO33
- net N$2: now also U$1.GPIO25; no longer U$1.GPIO26
Routing:
- net N$1: track 12.0 -> 1.80 mm
Changed lines of the file:
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@@
 </signal>
 <signal name="N$1">
-<contactref element="U$1" pad="GPIO33"/>
 <contactref element="SV2" pad="2"/>
-<wire x1="91.44" y1="44.45" x2="81.28" y2="44.45" width="0.254" layer="16"/>
 <wire x1="92.71" y1="45.72" x2="91.44" y2="44.45" width="0.254" layer="16"/>
+<contactref element="U$1" pad="GPIO32"/>
+<wire x1="81.28" y1="41.91" x2="91.44" y2="44.45" width="0" layer="19" extent="16-16"/>
 </signal>
 <signal name="N$3">
@@
 </signal>
 <signal name="N$2">
-<contactref element="U$1" pad="GPIO26"/>
+<contactref element="U$1" pad="GPIO25"/>
 </signal>
 </signals>
