File: accessControl.sch (EAGLE design)
At the start: 11 parts

Commit message: esp32 code
Parts:
- added U$2: DS3231, DS3231:DS3231
Connections:
- new net N$4: G1.-, G2.+
- new net N$5: G2.-, G3.+
- new net N$6: G3.-, G4.+
- new net N$8: U$1.GPIO22, U$2.SCL1
- new net N$9: U$1.GPIO21, U$2.SDA1
- net +3V3: now also U$2.VCC1
- net +5V: no longer G2.+, G3.+, G4.+
- net GND: now also U$2.GND1; no longer G1.-, G2.-, G3.-
- net N$1: now also U$1.GPIO32; no longer U$1.GPIO33
- net N$2: now also U$1.GPIO25; no longer U$1.GPIO26
Other:
- moved on the sheet: G1, G2, G3, G4
Changed lines of the file:
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@@
 <part name="GND4" library="supply1" library_urn="urn:adsk.eagle:library:371" deviceset="GND" device=""/>
 <part name="GND5" library="supply1" library_urn="urn:adsk.eagle:library:371" deviceset="GND" device=""/>
+<part name="U$2" library="DS3231" deviceset="DS3231" device=""/>
+<part name="+3V1" library="supply1" library_urn="urn:adsk.eagle:library:371" deviceset="+3V3" device=""/>
 </parts>
 <sheets>
@@
 <instances>
 <instance part="U$1" gate="G$1" x="48.26" y="25.4" smashed="yes"/>
-<instance part="G1" gate="1" x="-27.94" y="60.96" smashed="yes">
-<attribute name="NAME" x="-30.48" y="64.135" size="1.778" layer="95"/>
-<attribute name="VALUE" x="-30.48" y="55.88" size="1.778" layer="96"/>
-</instance>
-<instance part="G2" gate="1" x="-27.94" y="50.8" smashed="yes">
-<attribute name="NAME" x="-30.48" y="53.975" size="1.778" layer="95"/>
-<attribute name="VALUE" x="-30.48" y="45.72" size="1.778" layer="96"/>
-</instance>
-<instance part="G3" gate="1" x="-27.94" y="40.64" smashed="yes">
-<attribute name="NAME" x="-30.48" y="43.815" size="1.778" layer="95"/>
-<attribute name="VALUE" x="-30.48" y="35.56" size="1.778" layer="96"/>
-</instance>
-<instance part="G4" gate="1" x="-27.94" y="30.48" smashed="yes">
-<attribute name="NAME" x="-30.48" y="33.655" size="1.778" layer="95"/>
-<attribute name="VALUE" x="-30.48" y="25.4" size="1.778" layer="96"/>
-</instance>
-<instance part="GND1" gate="1" x="-33.02" y="17.78" smashed="yes">
-<attribute name="VALUE" x="-35.56" y="15.24" size="1.778" layer="96"/>
+<instance part="G1" gate="1" x="-17.78" y="66.04" smashed="yes" rot="R90">
+<attribute name="NAME" x="-20.955" y="63.5" size="1.778" layer="95" rot="R90"/>
+<attribute name="VALUE" x="-12.7" y="63.5" size="1.778" layer="96" rot="R90"/>
+</instance>
+<instance part="G2" gate="1" x="-17.78" y="55.88" smashed="yes" rot="R90">
+<attribute name="NAME" x="-20.955" y="53.34" size="1.778" layer="95" rot="R90"/>
+<attribute name="VALUE" x="-12.7" y="53.34" size="1.778" layer="96" rot="R90"/>
+</instance>
+<instance part="G3" gate="1" x="-17.78" y="45.72" smashed="yes" rot="R90">
+<attribute name="NAME" x="-20.955" y="43.18" size="1.778" layer="95" rot="R90"/>
+<attribute name="VALUE" x="-12.7" y="43.18" size="1.778" layer="96" rot="R90"/>
+</instance>
+<instance part="G4" gate="1" x="-17.78" y="35.56" smashed="yes" rot="R90">
+<attribute name="NAME" x="-20.955" y="33.02" size="1.778" layer="95" rot="R90"/>
+<attribute name="VALUE" x="-12.7" y="33.02" size="1.778" layer="96" rot="R90"/>
+</instance>
+<instance part="GND1" gate="1" x="-17.78" y="17.78" smashed="yes">
+<attribute name="VALUE" x="-20.32" y="15.24" size="1.778" layer="96"/>
 </instance>
 <instance part="GND2" gate="1" x="30.48" y="27.94" smashed="yes">
@@
 <attribute name="VALUE" x="12.7" y="55.88" size="1.778" layer="96"/>
 </instance>
-<instance part="P+1" gate="1" x="-22.86" y="71.12" smashed="yes">
-<attribute name="VALUE" x="-25.4" y="68.58" size="1.778" layer="96" rot="R270"/>
+<instance part="P+1" gate="1" x="-17.78" y="78.74" smashed="yes">
+<attribute name="VALUE" x="-20.32" y="76.2" size="1.778" layer="96" rot="R270"/>
 </instance>
 <instance part="P+2" gate="1" x="30.48" y="43.18" smashed="yes">
@@
 <instance part="GND5" gate="1" x="86.36" y="55.88" smashed="yes">
 <attribute name="VALUE" x="83.82" y="53.34" size="1.778" layer="96"/>
+</instance>
+<instance part="U$2" gate="G$1" x="147.32" y="68.58" smashed="yes" rot="R180">
+<attribute name="NAME" x="132.08" y="73.66" size="1.778" layer="94" rot="R270"/>
+<attribute name="VALUE" x="132.08" y="58.42" size="1.778" layer="94" rot="R270"/>
+</instance>
+<instance part="+3V1" gate="G$1" x="99.06" y="86.36" smashed="yes">
+<attribute name="VALUE" x="96.52" y="81.28" size="1.778" layer="96" rot="R90"/>
 </instance>
 </instances>
@@
 <net name="GND" class="4">
 <segment>
-<pinref part="G1" gate="1" pin="-"/>
-<pinref part="G2" gate="1" pin="-"/>
-<wire x1="-33.02" y1="60.96" x2="-33.02" y2="50.8" width="0.1524" layer="91"/>
-<pinref part="G3" gate="1" pin="-"/>
-<wire x1="-33.02" y1="50.8" x2="-33.02" y2="40.64" width="0.1524" layer="91"/>
-<junction x="-33.02" y="50.8"/>
 <pinref part="G4" gate="1" pin="-"/>
-<wire x1="-33.02" y1="40.64" x2="-33.02" y2="30.48" width="0.1524" layer="91"/>
-<junction x="-33.02" y="40.64"/>
-<wire x1="-33.02" y1="30.48" x2="-33.02" y2="20.32" width="0.1524" layer="91"/>
-<junction x="-33.02" y="30.48"/>
+<wire x1="-17.78" y1="30.48" x2="-17.78" y2="20.32" width="0.1524" layer="91"/>
 <pinref part="GND1" gate="1" pin="GND"/>
-<wire x1="-33.02" y1="20.32" x2="-33.02" y2="17.78" width="0.1524" layer="91"/>
-<junction x="-33.02" y="20.32"/>
+<wire x1="-17.78" y1="20.32" x2="-17.78" y2="17.78" width="0.1524" layer="91"/>
+<junction x="-17.78" y="20.32"/>
 </segment>
 <segment>
@@
 <pinref part="GND6" gate="1" pin="GND"/>
 <wire x1="78.74" y1="73.66" x2="88.9" y2="73.66" width="0.1524" layer="91"/>
+<pinref part="U$2" gate="G$1" pin="GND1"/>
+<wire x1="88.9" y1="73.66" x2="106.68" y2="73.66" width="0.1524" layer="91"/>
+<junction x="88.9" y="73.66"/>
 </segment>
 <segment>
@@
 </net>
 <net name="+5V" class="1">
-<segment>
-<pinref part="G1" gate="1" pin="+"/>
-<pinref part="G2" gate="1" pin="+"/>
-<wire x1="-22.86" y1="60.96" x2="-22.86" y2="50.8" width="0.1524" layer="91"/>
-<pinref part="G3" gate="1" pin="+"/>
-<wire x1="-22.86" y1="50.8" x2="-22.86" y2="40.64" width="0.1524" layer="91"/>
-<junction x="-22.86" y="50.8"/>
-<pinref part="G4" gate="1" pin="+"/>
-<wire x1="-22.86" y1="40.64" x2="-22.86" y2="30.48" width="0.1524" layer="91"/>
-<junction x="-22.86" y="40.64"/>
-<wire x1="-22.86" y1="60.96" x2="-22.86" y2="68.58" width="0.1524" layer="91"/>
-<junction x="-22.86" y="60.96"/>
-<pinref part="P+1" gate="1" pin="+5V"/>
-</segment>
 <segment>
 <wire x1="30.48" y1="35.56" x2="30.48" y2="38.1" width="0.1524" layer="91"/>
@@
 <wire x1="45.72" y1="27.94" x2="48.26" y2="27.94" width="0.1524" layer="91"/>
 </segment>
+<segment>
+<pinref part="G1" gate="1" pin="+"/>
+<pinref part="P+1" gate="1" pin="+5V"/>
+<wire x1="-17.78" y1="71.12" x2="-17.78" y2="76.2" width="0.1524" layer="91"/>
+</segment>
 </net>
 <net name="+3V3" class="3">
@@
 <junction x="43.18" y="73.66"/>
 </segment>
+<segment>
+<pinref part="U$2" gate="G$1" pin="VCC1"/>
+<wire x1="106.68" y1="68.58" x2="99.06" y2="68.58" width="0.1524" layer="91"/>
+<wire x1="99.06" y1="68.58" x2="99.06" y2="83.82" width="0.1524" layer="91"/>
+<pinref part="+3V1" gate="G$1" pin="+3V3"/>
+</segment>
 </net>
 <net name="N$1" class="0">
 <segment>
-<pinref part="U$1" gate="G$1" pin="GPIO33"/>
-<wire x1="48.26" y1="55.88" x2="22.86" y2="55.88" width="0.1524" layer="91"/>
-<wire x1="22.86" y1="55.88" x2="22.86" y2="68.58" width="0.1524" layer="91"/>
 <pinref part="SV2" gate="G$1" pin="2"/>
+<wire x1="22.86" y1="58.42" x2="22.86" y2="68.58" width="0.1524" layer="91"/>
 <wire x1="22.86" y1="68.58" x2="7.62" y2="68.58" width="0.1524" layer="91"/>
+<pinref part="U$1" gate="G$1" pin="GPIO32"/>
+<wire x1="48.26" y1="58.42" x2="22.86" y2="58.42" width="0.1524" layer="91"/>
 </segment>
 </net>
@@
 <net name="N$2" class="0">
 <segment>
+<pinref part="U$1" gate="G$1" pin="GPIO25"/>
 <pinref part="R2" gate="G$1" pin="2"/>
-<pinref part="U$1" gate="G$1" pin="GPIO26"/>
-<wire x1="40.64" y1="50.8" x2="48.26" y2="50.8" width="0.1524" layer="91"/>
-</segment>
-</net>
+<wire x1="48.26" y1="53.34" x2="40.64" y2="53.34" width="0.1524" layer="91"/>
+<wire x1="40.64" y1="53.34" x2="40.64" y2="50.8" width="0.1524" layer="91"/>
+</segment>
+</net>
+<net name="N$4" class="0">
+<segment>
+<pinref part="G1" gate="1" pin="-"/>
+<pinref part="G2" gate="1" pin="+"/>
+</segment>
+</net>
+<net name="N$5" class="0">
+<segment>
+<pinref part="G2" gate="1" pin="-"/>
+<pinref part="G3" gate="1" pin="+"/>
+</segment>
+</net>
+<net name="N$6" class="0">
+<segment>
+<pinref part="G4" gate="1" pin="+"/>
+<pinref part="G3" gate="1" pin="-"/>
+</segment>
+</net>
+<net name="N$8" class="0">
+<segment>
+<pinref part="U$2" gate="G$1" pin="SCL1"/>
+<wire x1="106.68" y1="58.42" x2="96.52" y2="58.42" width="0.1524" layer="91"/>
+<wire x1="96.52" y1="58.42" x2="96.52" y2="68.58" width="0.1524" layer="91"/>
+<pinref part="U$1" gate="G$1" pin="GPIO22"/>
+<wire x1="96.52" y1="68.58" x2="78.74" y2="68.58" width="0.1524" layer="91"/>
+</segment>
+</net>
+<net name="N$9" class="0">
+<segment>
+<pinref part="U$2" gate="G$1" pin="SDA1"/>
+<wire x1="106.68" y1="63.5" x2="88.9" y2="63.5" width="0.1524" layer="91"/>
+<wire x1="88.9" y1="63.5" x2="88.9" y2="60.96" width="0.1524" layer="91"/>
+<pinref part="U$1" gate="G$1" pin="GPIO21"/>
+<wire x1="88.9" y1="60.96" x2="78.74" y2="60.96" width="0.1524" layer="91"/>
+</segment>
+</net>
